File: hardware/watch.kicad_pcb (KiCad board)
At the start: 4 copper layers, 39.1 x 36.2 mm, 77 parts, among them J1 DX07S016JA1R1500, J601 SWD, Q1 DMN6140L, Q401 DMP2110UW-7, Q701 DMP2110UW-7, SW601 SW_Push, SW602 SW_Push, U12 TCPP01-M12, U201 KCSA02-105, U202 STP08DP05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

Commit message: finished routing
Parts:
- C1, C301, D1, D2, F301, FB301, Q1, R10, R11, U12: moved to F.Cu
- C503, C504, U502: moved to B.Cu
- moved C601 51.0 mm to (159.1, 130.5), turned to 0 degrees
- moved C602 46.9 mm to (159.1, 128.0), turned to 0 degrees
- moved Y601 45.8 mm to (156.3, 129.3), turned to 270 degrees
- moved R602 44.7 mm to (152.9, 131.1), turned to 180 degrees
- moved J601 43.1 mm to (143.4, 130.5), turned to 0 degrees
- moved R405 41.2 mm to (159.8, 125.8), turned to 0 degrees
- moved R404 39.1 mm to (159.8, 124.2), turned to 180 degrees
- moved U601 35.8 mm to (150.8, 126.8), turned to 180 degrees
- moved C606 35.4 mm to (149.8, 131.1), turned to 180 degrees
- moved C607 34.4 mm to (146.2, 127.2), turned to 90 degrees
- moved C605 29.4 mm to (144.4, 127.1), turned to 90 degrees
- moved C504 24.2 mm to (155.9, 116.1)
- moved U502 18.7 mm to (155.9, 113.3), turned to 270 degrees
- moved U12 15.0 mm to (125.8, 129.3), turned to 90 degrees
- moved C503 13.1 mm to (155.9, 110.5)
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Connections:
- C603 pad 1: /Microcontroller Circuitry/SW1 -> /Microcontroller Circuitry/SW2
- C604 pad 1: /Microcontroller Circuitry/SW2 -> /Microcontroller Circuitry/SW1
- R601 pad 1: /Microcontroller Circuitry/SW1 -> /Microcontroller Circuitry/SW2
- R603 pad 1: /Microcontroller Circuitry/SW2 -> /Microcontroller Circuitry/SW1
Routing:
- net GND: track 190.7 -> 115.5 mm, vias 1 -> 0
- net /Display/CLK: track 0.00 -> 60.3 mm, vias 0 -> 5
- net +3V3: track 37.0 -> 95.0 mm, vias 0 -> 1
- net /Display/LE: track 0.00 -> 58.0 mm, vias 0 -> 5
- net /Microcontroller Circuitry/MOSI: track 0.00 -> 56.3 mm, vias 0 -> 2
- net /Microcontroller Circuitry/SW2: track 0.00 -> 54.4 mm, vias 0 -> 2
- net /Display/OE: track 0.00 -> 54.1 mm, vias 0 -> 5
- net /Microcontroller Circuitry/SW1: track 0.00 -> 35.2 mm, vias 0 -> 2
- net /USB/RX: track 0.00 -> 32.5 mm, vias 0 -> 2
- net /Microcontroller Circuitry/RX: track 0.00 -> 27.8 mm, vias 0 -> 2
- net /USB/CTS: track 0.00 -> 27.6 mm, vias 0 -> 2
- net /USB Protection Circuits/V_BUS_CTRL: track 24.8 -> 6.83 mm
- net Net-(D1-Pad1): track 25.3 -> 7.52 mm
- net /Battery Charger/VBAT: track 9.05 -> 23.8 mm, vias 0 -> 2
- net /Microcontroller Circuitry/NRST: track 0.00 -> 14.6 mm, vias 0 -> 2
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- added copper zone on B.Cu, net GND
- added copper zone on F.Cu, net GND
- added copper zone on In1.Cu, net GND
Other:
- board size 39.1 x 36.2 mm -> 39.1 x 36.1 mm

Commit message: calc current consumption
Parts:
- R201, R202, R203, R204: value 2k -> 6k8
- R501: value 10k -> 1k
Connections:
- U501 pad 2: GND -> Net-(U501-Pad2)
- U501 pad 3: Net-(U501-Pad3) -> GND
Routing:
- net GND: track 115.5 -> 114.5 mm
