File: hardware/Microcontroller.sch (KiCad schematic (older format))
At the start: 15 parts, among them J601 SWD, SW601 SW_Push, SW602 SW_Push, U601 STM32L011F4Px, Y601 32kHz

Commit message: wip hw
Parts:
- C601, C602, C603, C604, C606, C607: footprint Capacitor_SMD:C_0603_1608Metric_Pad1.05x0.95mm_HandSolder -> Capacitor_SMD:C_0603_1608Metric
- C605: footprint Capacitor_SMD:C_0603_1608Metric_Pad1.05x0.95mm_HandSolder -> Capacitor_SMD:C_0805_2012Metric
- R601, R602, R603: footprint Resistor_SMD:R_0603_1608Metric_Pad1.05x0.95mm_HandSolder -> Resistor_SMD:R_0603_1608Metric
Changed lines of the file:
@@
 F 0 "C605" H 3792 1646 50  0000 L CNN
 F 1 "10u" H 3792 1555 50  0000 L CNN
-F 2 "Capacitor_SMD:C_0603_1608Metric_Pad1.05x0.95mm_HandSolder" H 3700 1600 50  0001 C CNN
+F 2 "Capacitor_SMD:C_0805_2012Metric" H 3700 1600 50  0001 C CNN
 F 3 "https://www.mouser.at/datasheet/2/585/MLCC-1837944.pdf" H 3700 1600 50  0001 C CNN
 F 4 "https://www.mouser.at/ProductDetail/187-CL10B106MQ8NRNC" H 3700 1600 50  0001 C CNN "Order"
@@
 F 0 "C606" H 4242 1646 50  0000 L CNN
 F 1 "100n" H 4242 1555 50  0000 L CNN
-F 2 "Capacitor_SMD:C_0603_1608Metric_Pad1.05x0.95mm_HandSolder" H 4150 1600 50  0001 C CNN
+F 2 "Capacitor_SMD:C_0603_1608Metric" H 4150 1600 50  0001 C CNN
 F 3 "https://www.mouser.at/datasheet/2/212/KEM_C1002_X7R_SMD-1102033.pdf" H 4150 1600 50  0001 C CNN
 F 4 "https://www.mouser.at/ProductDetail/80-C0603C104M4R" H 4150 1600 50  0001 C CNN "Order"
@@
 F 0 "C601" H 692 2496 50  0000 L CNN
 F 1 "12p" H 692 2405 50  0000 L CNN
-F 2 "Capacitor_SMD:C_0603_1608Metric_Pad1.05x0.95mm_HandSolder" H 600 2450 50  0001 C CNN
+F 2 "Capacitor_SMD:C_0603_1608Metric" H 600 2450 50  0001 C CNN
 F 3 "https://www.mouser.at/datasheet/2/212/KEM_C1007_X8R_ULTRA_150C_SMD-1102703.pdf" H 600 2450 50  0001 C CNN
 F 4 "https://www.mouser.at/ProductDetail/80-C0603C120K5HACTU" H 600 2450 50  0001 C CNN "Order"
@@
 F 0 "C602" H 1392 2496 50  0000 L CNN
 F 1 "12p" H 1392 2405 50  0000 L CNN
-F 2 "Capacitor_SMD:C_0603_1608Metric_Pad1.05x0.95mm_HandSolder" H 1300 2450 50  0001 C CNN
+F 2 "Capacitor_SMD:C_0603_1608Metric" H 1300 2450 50  0001 C CNN
 F 3 "https://www.mouser.at/datasheet/2/212/KEM_C1007_X8R_ULTRA_150C_SMD-1102703.pdf" H 1300 2450 50  0001 C CNN
 F 4 "https://www.mouser.at/ProductDetail/80-C0603C120K5HACTU" H 1300 2450 50  0001 C CNN "Order"
@@
 F 0 "C607" H 4692 1646 50  0000 L CNN
 F 1 "100n" H 4692 1555 50  0000 L CNN
-F 2 "Capacitor_SMD:C_0603_1608Metric_Pad1.05x0.95mm_HandSolder" H 4600 1600 50  0001 C CNN
+F 2 "Capacitor_SMD:C_0603_1608Metric" H 4600 1600 50  0001 C CNN
 F 3 "https://www.mouser.at/datasheet/2/212/KEM_C1002_X7R_SMD-1102033.pdf" H 4600 1600 50  0001 C CNN
 F 4 "https://www.mouser.at/ProductDetail/80-C0603C104M4R" H 4600 1600 50  0001 C CNN "Order"
@@
 F 0 "C603" H 1542 4246 50  0000 L CNN
 F 1 "100n" H 1542 4155 50  0000 L CNN
-F 2 "Capacitor_SMD:C_0603_1608Metric_Pad1.05x0.95mm_HandSolder" H 1450 4200 50  0001 C CNN
+F 2 "Capacitor_SMD:C_0603_1608Metric" H 1450 4200 50  0001 C CNN
 F 3 "https://www.mouser.at/datasheet/2/212/KEM_C1002_X7R_SMD-1102033.pdf" H 1450 4200 50  0001 C CNN
 F 4 "https://www.mouser.at/ProductDetail/80-C0603C104M4R" H 1450 4200 50  0001 C CNN "Order"
@@
 F 0 "C604" H 2742 4246 50  0000 L CNN
 F 1 "100n" H 2742 4155 50  0000 L CNN
-F 2 "Capacitor_SMD:C_0603_1608Metric_Pad1.05x0.95mm_HandSolder" H 2650 4200 50  0001 C CNN
+F 2 "Capacitor_SMD:C_0603_1608Metric" H 2650 4200 50  0001 C CNN
 F 3 "https://www.mouser.at/datasheet/2/212/KEM_C1002_X7R_SMD-1102033.pdf" H 2650 4200 50  0001 C CNN
 F 4 "https://www.mouser.at/ProductDetail/80-C0603C104M4R" H 2650 4200 50  0001 C CNN "Order"
@@
 F 0 "R602" H 1609 3046 50  0000 L CNN
 F 1 "100k" H 1609 2955 50  0000 L CNN
-F 2 "Resistor_SMD:R_0603_1608Metric_Pad1.05x0.95mm_HandSolder" H 1550 3000 50  0001 C CNN
+F 2 "Resistor_SMD:R_0603_1608Metric" H 1550 3000 50  0001 C CNN
 F 3 "https://www.mouser.at/datasheet/2/418/5/NG_DS_9-1773463-9_A-1358566.pdf" H 1550 3000 50  0001 C CNN
 F 4 "https://www.mouser.at/ProductDetail/279-CRGP0603F100K" H 1550 3000 50  0001 C CNN "Order"
@@
 F 0 "R601" V 1004 3950 50  0000 C CNN
 F 1 "R_Small" V 1095 3950 50  0000 C CNN
-F 2 "Resistor_SMD:R_0603_1608Metric_Pad1.05x0.95mm_HandSolder" H 1200 3950 50  0001 C CNN
+F 2 "Resistor_SMD:R_0603_1608Metric" H 1200 3950 50  0001 C CNN
 F 3 "~" H 1200 3950 50  0001 C CNN
 	1    1200 3950
@@
 F 0 "R603" V 2204 3950 50  0000 C CNN
 F 1 "R_Small" V 2295 3950 50  0000 C CNN
-F 2 "Resistor_SMD:R_0603_1608Metric_Pad1.05x0.95mm_HandSolder" H 2400 3950 50  0001 C CNN
+F 2 "Resistor_SMD:R_0603_1608Metric" H 2400 3950 50  0001 C CNN
 F 3 "~" H 2400 3950 50  0001 C CNN
 	1    2400 3950

Commit message: finished routing
Connections:
- net SW1: now also C604.1, R603.1; no longer C603.1, R601.1
- net SW2: now also C603.1, R601.1; no longer C604.1, R603.1
Changed lines of the file:
@@
 Wire Wire Line
 	2150 4450 2400 4450
-Text Label 2850 3950 2    50   ~ 0
+Text Label 1650 3950 2    50   ~ 0
 SW2
 Wire Wire Line
@@
 	0    1    1    0
 $EndComp
-Text Label 1650 3950 2    50   ~ 0
+Text Label 2850 3950 2    50   ~ 0
 SW1
 Wire Wire Line

Commit message: calc current consumption
Parts:
- R601, R603: value R_Small -> 1k
Changed lines of the file:
@@
 P 1200 3950
 F 0 "R601" V 1004 3950 50  0000 C CNN
-F 1 "R_Small" V 1095 3950 50  0000 C CNN
+F 1 "1k" V 1095 3950 50  0000 C CNN
 F 2 "Resistor_SMD:R_0603_1608Metric" H 1200 3950 50  0001 C CNN
 F 3 "~" H 1200 3950 50  0001 C CNN
@@
 P 2400 3950
 F 0 "R603" V 2204 3950 50  0000 C CNN
-F 1 "R_Small" V 2295 3950 50  0000 C CNN
+F 1 "1k" V 2295 3950 50  0000 C CNN
 F 2 "Resistor_SMD:R_0603_1608Metric" H 2400 3950 50  0001 C CNN
 F 3 "~" H 2400 3950 50  0001 C CNN

Commit message: added powerflags
Connections:
- no-connect marks 0 -> 1
Changed lines of the file:
@@
 Wire Wire Line
 	3950 2900 4000 2900
+NoConn ~ 4500 2900
 $EndSCHEMATC
