File: hardware/Power_Selection.sch (KiCad schematic (older format))
At the start: 7 parts, among them U501 TPS2115A-Q1, U502 TLV70033_SOT23-5

Commit message: wip hw
Parts:
- C501, C502, C503, C504: footprint Capacitor_SMD:C_0603_1608Metric_Pad1.05x0.95mm_HandSolder -> Capacitor_SMD:C_0603_1608Metric
- R501: footprint Resistor_SMD:R_0603_1608Metric_Pad1.05x0.95mm_HandSolder -> Resistor_SMD:R_0603_1608Metric
Changed lines of the file:
@@
 F 0 "C503" H 3342 2246 50  0000 L CNN
 F 1 "1u" H 3342 2155 50  0000 L CNN
-F 2 "Capacitor_SMD:C_0603_1608Metric_Pad1.05x0.95mm_HandSolder" H 3250 2200 50  0001 C CNN
+F 2 "Capacitor_SMD:C_0603_1608Metric" H 3250 2200 50  0001 C CNN
 F 3 "https://www.mouser.at/datasheet/2/585/MLCC-1837944.pdf" H 3250 2200 50  0001 C CNN
 F 4 "https://www.mouser.at/ProductDetail/187-CL10B105MO8NNWC" H 3250 2200 50  0001 C CNN "Order"
@@
 F 0 "C504" H 4492 2246 50  0000 L CNN
 F 1 "1u" H 4492 2155 50  0000 L CNN
-F 2 "Capacitor_SMD:C_0603_1608Metric_Pad1.05x0.95mm_HandSolder" H 4400 2200 50  0001 C CNN
+F 2 "Capacitor_SMD:C_0603_1608Metric" H 4400 2200 50  0001 C CNN
 F 3 "https://www.mouser.at/datasheet/2/585/MLCC-1837944.pdf" H 4400 2200 50  0001 C CNN
 F 4 "https://www.mouser.at/ProductDetail/187-CL10B105MO8NNWC" H 4400 2200 50  0001 C CNN "Order"
@@
 F 0 "R501" H 2059 2646 50  0000 L CNN
 F 1 "10k" H 2059 2555 50  0000 L CNN
-F 2 "Resistor_SMD:R_0603_1608Metric_Pad1.05x0.95mm_HandSolder" H 2000 2600 50  0001 C CNN
+F 2 "Resistor_SMD:R_0603_1608Metric" H 2000 2600 50  0001 C CNN
 F 3 "~" H 2000 2600 50  0001 C CNN
 F 4 "" H 2000 2600 50  0001 C CNN "Order"
@@
 F 0 "C501" H 1092 2296 50  0000 L CNN
 F 1 "100n" H 1092 2205 50  0000 L CNN
-F 2 "Capacitor_SMD:C_0603_1608Metric_Pad1.05x0.95mm_HandSolder" H 1000 2250 50  0001 C CNN
+F 2 "Capacitor_SMD:C_0603_1608Metric" H 1000 2250 50  0001 C CNN
 F 3 "https://www.mouser.at/datasheet/2/212/KEM_C1002_X7R_SMD-1102033.pdf" H 1000 2250 50  0001 C CNN
 F 4 "https://www.mouser.at/ProductDetail/80-C0603C104M4R" H 1000 2250 50  0001 C CNN "Order"
@@
 F 0 "C502" H 1542 2296 50  0000 L CNN
 F 1 "100n" H 1542 2205 50  0000 L CNN
-F 2 "Capacitor_SMD:C_0603_1608Metric_Pad1.05x0.95mm_HandSolder" H 1450 2250 50  0001 C CNN
+F 2 "Capacitor_SMD:C_0603_1608Metric" H 1450 2250 50  0001 C CNN
 F 3 "https://www.mouser.at/datasheet/2/212/KEM_C1002_X7R_SMD-1102033.pdf" H 1450 2250 50  0001 C CNN
 F 4 "https://www.mouser.at/ProductDetail/80-C0603C104M4R" H 1450 2250 50  0001 C CNN "Order"

Commit message: calc current consumption
Parts:
- R501: value 10k -> 1k
Connections:
- net GND: now also U501.3 (D1); no longer U501.2 (D0)
Changed lines of the file:
@@
 AR Path="/605CEFBE/605D36D8" Ref="R501"  Part="1"
 F 0 "R501" H 2059 2646 50  0000 L CNN
-F 1 "10k" H 2059 2555 50  0000 L CNN
+F 1 "1k" H 2059 2555 50  0000 L CNN
 F 2 "Resistor_SMD:R_0603_1608Metric" H 2000 2600 50  0001 C CNN
 F 3 "~" H 2000 2600 50  0001 C CNN
@@
 	1    0    0    -1
 $EndComp
-Wire Wire Line
-	2050 2350 1850 2350
-Wire Wire Line
-	1850 2350 1850 2700
 $Comp
 L power:GND #PWR?
@@
 	1    0    0    -1
 $EndComp
-NoConn ~ 2050 2250
 Wire Wire Line
 	3250 2300 3250 2450
@@
 Wire Wire Line
 	3350 1600 3250 1600
+NoConn ~ 2050 2350
+Wire Wire Line
+	1850 2250 2050 2250
+Wire Wire Line
+	1850 2250 1850 2700
 $EndSCHEMATC

Commit message: added powerflags
Connections:
- no-connect marks 1 -> 2
Changed lines of the file:
@@
 Wire Wire Line
 	1850 2250 1850 2700
+NoConn ~ 2750 2200
 $EndSCHEMATC
