File: hardware/Power_Selection.sch (KiCad schematic (older format))
At the start: 7 parts, among them U501 TPS2115A-Q1, U502 TLV70033_SOT23-5

Commit message: added order references to parts
Parts:
- R501: Manufacturer (none) -> TE Connectivity / Holsworthy; Order (none) -> https://www.mouser.at/ProductDetail/TE-Connectivity-Holswor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
- U501: Manufacturer (none) -> Texas Instruments; Order (none) -> https://www.mouser.at/ProductDetail/Texas-Instruments/TPS21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
Changed lines of the file:
@@
 F 2 "watch:TSSOP-8_3x6.4_P0.65mm" H 3300 3050 50  0001 C CNN
 F 3 "" H 3300 3050 50  0001 C CNN
+F 4 "Texas Instruments" H 2400 2200 50  0001 C CNN "Manufacturer"
+F 5 "https://www.mouser.at/ProductDetail/Texas-Instruments/TPS2115AIPWRQ1?qs=%2Fha2pyFadugZrMbQPJQt%252BSVlkr%252BjGGlgJkJQJe24P%252BubSh98JtzVLQ%3D%3D" H 2400 2200 50  0001 C CNN "Order"
 	1    2400 2200
 	1    0    0    -1
@@
 F 2 "Resistor_SMD:R_0603_1608Metric" H 2000 2600 50  0001 C CNN
 F 3 "~" H 2000 2600 50  0001 C CNN
-F 4 "" H 2000 2600 50  0001 C CNN "Order"
+F 4 "https://www.mouser.at/ProductDetail/TE-Connectivity-Holsworthy/CRGP0603F1K0?qs=sGAEpiMZZMtlubZbdhIBIOInyB5Ysv8sRTd2oyB6aAs%3D" H 2000 2600 50  0001 C CNN "Order"
+F 5 "TE Connectivity / Holsworthy" H 2000 2600 50  0001 C CNN "Manufacturer"
 	1    2000 2600
 	1    0    0    -1

Commit message: modified bom
Parts:
- C501, C502: MNR (none) -> C0603C104M4RACTU
- C503, C504: MNR (none) -> CL10B105MO8NNWC
- R501: MNR (none) -> CRGP0603F1K0
- U501: MNR (none) -> TPS2115AIPWRQ1
- U502: MNR (none) -> TLV70033DDCR
Changed lines of the file:
@@
 F 4 "https://www.mouser.at/ProductDetail/187-CL10B105MO8NNWC" H 3250 2200 50  0001 C CNN "Order"
 F 5 "Samsung Electro-Mechanics" H 3250 2200 50  0001 C CNN "Manufacturer"
+F 6 "CL10B105MO8NNWC" H 3250 2200 50  0001 C CNN "MNR"
 	1    3250 2200
 	1    0    0    -1
@@
 F 4 "https://www.mouser.at/ProductDetail/187-CL10B105MO8NNWC" H 4400 2200 50  0001 C CNN "Order"
 F 5 "Samsung Electro-Mechanics" H 4400 2200 50  0001 C CNN "Manufacturer"
+F 6 "CL10B105MO8NNWC" H 4400 2200 50  0001 C CNN "MNR"
 	1    4400 2200
 	1    0    0    -1
@@
 F 4 "https://www.mouser.at/ProductDetail/595-TLV70033DDCR" H 3850 2100 50  0001 C CNN "Order"
 F 5 "Texas Instruments" H 3850 2100 50  0001 C CNN "Manufacturer"
+F 6 "TLV70033DDCR" H 3850 2100 50  0001 C CNN "MNR"
 	1    3850 2100
 	1    0    0    -1
@@
 F 4 "Texas Instruments" H 2400 2200 50  0001 C CNN "Manufacturer"
 F 5 "https://www.mouser.at/ProductDetail/Texas-Instruments/TPS2115AIPWRQ1?qs=%2Fha2pyFadugZrMbQPJQt%252BSVlkr%252BjGGlgJkJQJe24P%252BubSh98JtzVLQ%3D%3D" H 2400 2200 50  0001 C CNN "Order"
+F 6 "TPS2115AIPWRQ1" H 2400 2200 50  0001 C CNN "MNR"
 	1    2400 2200
 	1    0    0    -1
@@
 F 4 "https://www.mouser.at/ProductDetail/TE-Connectivity-Holsworthy/CRGP0603F1K0?qs=sGAEpiMZZMtlubZbdhIBIOInyB5Ysv8sRTd2oyB6aAs%3D" H 2000 2600 50  0001 C CNN "Order"
 F 5 "TE Connectivity / Holsworthy" H 2000 2600 50  0001 C CNN "Manufacturer"
+F 6 "CRGP0603F1K0" H 2000 2600 50  0001 C CNN "MNR"
 	1    2000 2600
 	1    0    0    -1
@@
 F 4 "https://www.mouser.at/ProductDetail/80-C0603C104M4R" H 1000 2250 50  0001 C CNN "Order"
 F 5 "KEMET" H 1000 2250 50  0001 C CNN "Manufacturer"
+F 6 "C0603C104M4RACTU" H 1000 2250 50  0001 C CNN "MNR"
 	1    1000 2250
 	1    0    0    -1
@@
 F 4 "https://www.mouser.at/ProductDetail/80-C0603C104M4R" H 1450 2250 50  0001 C CNN "Order"
 F 5 "KEMET" H 1450 2250 50  0001 C CNN "Manufacturer"
+F 6 "C0603C104M4RACTU" H 1450 2250 50  0001 C CNN "MNR"
 	1    1450 2250
 	1    0    0    -1

Commit message: Updated to KiCad v6.0
Parts:
- added Q2: DMP2110UW-7, Package_TO_SOT_SMD:SOT-323_SC-70, symbol Device:Q_PMOS_GSD
- added R1: 1k, Resistor_SMD:R_0603_1608Metric, symbol Device:R_Small
Connections:
- net V_DISP: now also Q2.3 (D); no longer C503.1, U501.7 (OUT), U502.1 (IN), U502.3 (EN)
- net 3V3 renamed VuC
- new net: C503.1, Q2.2 (S), U501.7 (OUT), U502.1 (IN), U502.3 (EN)
- new net: Q2.1 (G), R1.1
- new net LED_CTRL: R1.2
Changed lines of the file:
@@
 Wire Wire Line
 	750  2050 1450 2050
-Text HLabel 3350 1600 2    50   Output ~ 0
+Text HLabel 5700 1600 2    50   Output ~ 0
 V_DISP
 Text HLabel 4650 2000 2    50   Output ~ 0
-3V3
+VuC
 Wire Wire Line
 	4400 2000 4650 2000
 Wire Wire Line
 	3250 1600 3250 2000
-Wire Wire Line
-	3350 1600 3250 1600
 NoConn ~ 2050 2350
 Wire Wire Line
@@
 	1850 2250 1850 2700
 NoConn ~ 2750 2200
+Text HLabel 5350 2200 0    50   Input ~ 0
+LED_CTRL
+$Comp
+L Device:Q_PMOS_GSD Q?
+U 1 1 61A64800
+P 5400 1700
+AR Path="/6063DAC2/61A64800" Ref="Q?"  Part="1"
+AR Path="/605CEFBE/61A64800" Ref="Q2"  Part="1"
+F 0 "Q2" V 5742 1700 50  0000 C CNN
+F 1 "DMP2110UW-7" V 5651 1700 50  0000 C CNN
+F 2 "Package_TO_SOT_SMD:SOT-323_SC-70" H 5600 1800 50  0001 C CNN
+F 3 "https://www.diodes.com/assets/Datasheets/DMP2110UW.pdf" H 5400 1700 50  0001 C CNN
+F 4 "Diodes Incorporated" H 5400 1700 50  0001 C CNN "Manufacturer"
+F 5 "https://www.mouser.at/ProductDetail/Diodes-Incorporated/DMP2110UW-7?qs=bZr6mbWTK5lZsAURvLPe3w%3D%3D" H 5400 1700 50  0001 C CNN "Order"
+F 6 "DMP2110UW-7" H 5400 1700 50  0001 C CNN "MNR"
+	1    5400 1700
+	0    1    -1   0
+$EndComp
+$Comp
+L Device:R_Small R?
+U 1 1 61A94055
+P 5400 2050
+AR Path="/61A94055" Ref="R?"  Part="1"
+AR Path="/605CEFBE/61A94055" Ref="R1"  Part="1"
+F 0 "R1" H 5459 2096 50  0000 L CNN
+F 1 "1k" H 5459 2005 50  0000 L CNN
+F 2 "Resistor_SMD:R_0603_1608Metric" H 5400 2050 50  0001 C CNN
+F 3 "~" H 5400 2050 50  0001 C CNN
+F 4 "https://www.mouser.at/ProductDetail/TE-Connectivity-Holsworthy/CRGP0603F1K0?qs=sGAEpiMZZMtlubZbdhIBIOInyB5Ysv8sRTd2oyB6aAs%3D" H 5400 2050 50  0001 C CNN "Order"
+F 5 "TE Connectivity / Holsworthy" H 5400 2050 50  0001 C CNN "Manufacturer"
+F 6 "CRGP0603F1K0" H 5400 2050 50  0001 C CNN "MNR"
+	1    5400 2050
+	1    0    0    -1
+$EndComp
+Wire Wire Line
+	5350 2200 5400 2200
+Wire Wire Line
+	5400 2200 5400 2150
+Wire Wire Line
+	5400 1950 5400 1900
+Wire Wire Line
+	5700 1600 5600 1600
+Wire Wire Line
+	3250 1600 5200 1600
 $EndSCHEMATC
