File: hardware/USB.sch (KiCad schematic (older format))
At the start: 13 parts, among them Q701 DMP2110UW-7, U701 FT230XQ

Commit message: wip hw
Parts:
- C701, C702, C704, C705, C706, C707: footprint Capacitor_SMD:C_0603_1608Metric_Pad1.05x0.95mm_HandSolder -> Capacitor_SMD:C_0603_1608Metric
- C703: footprint Capacitor_SMD:C_0603_1608Metric_Pad1.05x0.95mm_HandSolder -> Capacitor_SMD:C_0805_2012Metric
- Q701: footprint Package_TO_SOT_SMD:SOT-323_SC-70_Handsoldering -> Package_TO_SOT_SMD:SOT-323_SC-70
- R701, R702, R703, R704: footprint Resistor_SMD:R_0603_1608Metric_Pad1.05x0.95mm_HandSolder -> Resistor_SMD:R_0603_1608Metric
Connections:
- net CHIP_D-: now reaches R702.2, U701.6 (USBDP)
- net CHIP_D+: now reaches R701.2, U701.7 (USBDM)
Other:
- moved on the sheet: C701, C702, C704, R701, R702
Changed lines of the file:
@@
 Text HLabel 3700 1250 0    50   Input ~ 0
 VBUS
-Text HLabel 3450 2150 0    50   Input ~ 0
+Text HLabel 3100 2150 0    50   Input ~ 0
 D+
-Text HLabel 4000 2250 0    50   Input ~ 0
+Text HLabel 3650 2250 0    50   Input ~ 0
 D-
 $Comp
 L Device:C_Small C702
 U 1 1 60604C73
-P 3500 2300
-F 0 "C702" H 3592 2346 50  0000 L CNN
-F 1 "47p" H 3592 2255 50  0000 L CNN
-F 2 "Capacitor_SMD:C_0603_1608Metric_Pad1.05x0.95mm_HandSolder" H 3500 2300 50  0001 C CNN
-F 3 "~" H 3500 2300 50  0001 C CNN
-	1    3500 2300
+P 3150 2300
+F 0 "C702" H 3242 2346 50  0000 L CNN
+F 1 "47p" H 3242 2255 50  0000 L CNN
+F 2 "Capacitor_SMD:C_0603_1608Metric" H 3150 2300 50  0001 C CNN
+F 3 "~" H 3150 2300 50  0001 C CNN
+	1    3150 2300
 	1    0    0    -1
 $EndComp
@@
 L Device:C_Small C704
 U 1 1 60604FCD
-P 4050 2400
-F 0 "C704" H 4142 2446 50  0000 L CNN
-F 1 "47p" H 4142 2355 50  0000 L CNN
-F 2 "Capacitor_SMD:C_0603_1608Metric_Pad1.05x0.95mm_HandSolder" H 4050 2400 50  0001 C CNN
-F 3 "~" H 4050 2400 50  0001 C CNN
-	1    4050 2400
-	1    0    0    -1
-$EndComp
-Wire Wire Line
-	3450 2150 3500 2150
-Wire Wire Line
-	3500 2150 3500 2200
-Wire Wire Line
-	4050 2300 4050 2250
-Wire Wire Line
-	4050 2250 4000 2250
+P 3700 2400
+F 0 "C704" H 3792 2446 50  0000 L CNN
+F 1 "47p" H 3792 2355 50  0000 L CNN
+F 2 "Capacitor_SMD:C_0603_1608Metric" H 3700 2400 50  0001 C CNN
+F 3 "~" H 3700 2400 50  0001 C CNN
+	1    3700 2400
+	1    0    0    -1
+$EndComp
+Wire Wire Line
+	3100 2150 3150 2150
+Wire Wire Line
+	3150 2150 3150 2200
+Wire Wire Line
+	3700 2300 3700 2250
+Wire Wire Line
+	3700 2250 3650 2250
 $Comp
 L Interface_USB:FT230XQ U701
@@
 L Device:R_Small R701
 U 1 1 60606806
-P 4400 2150
-F 0 "R701" V 4450 2300 50  0000 C CNN
-F 1 "27R" V 4450 2000 50  0000 C CNN
-F 2 "Resistor_SMD:R_0603_1608Metric_Pad1.05x0.95mm_HandSolder" H 4400 2150 50  0001 C CNN
-F 3 "~" H 4400 2150 50  0001 C CNN
-	1    4400 2150
+P 4050 2150
+F 0 "R701" V 4100 2300 50  0000 C CNN
+F 1 "27R" V 4100 2000 50  0000 C CNN
+F 2 "Resistor_SMD:R_0603_1608Metric" H 4050 2150 50  0001 C CNN
+F 3 "~" H 4050 2150 50  0001 C CNN
+	1    4050 2150
 	0    -1   -1   0
 $EndComp
@@
 L Device:R_Small R702
 U 1 1 6060717E
-P 4400 2250
-F 0 "R702" V 4450 2400 50  0000 C CNN
-F 1 "27R" V 4450 2100 50  0000 C CNN
-F 2 "Resistor_SMD:R_0603_1608Metric_Pad1.05x0.95mm_HandSolder" H 4400 2250 50  0001 C CNN
-F 3 "~" H 4400 2250 50  0001 C CNN
-	1    4400 2250
+P 4050 2250
+F 0 "R702" V 4100 2400 50  0000 C CNN
+F 1 "27R" V 4100 2100 50  0000 C CNN
+F 2 "Resistor_SMD:R_0603_1608Metric" H 4050 2250 50  0001 C CNN
+F 3 "~" H 4050 2250 50  0001 C CNN
+	1    4050 2250
 	0    -1   -1   0
 $EndComp
 Wire Wire Line
-	4500 2150 4650 2150
-Wire Wire Line
-	4500 2250 4650 2250
-Wire Wire Line
-	3500 2150 4300 2150
-Connection ~ 3500 2150
-Wire Wire Line
-	4300 2250 4050 2250
-Connection ~ 4050 2250
+	3150 2150 3950 2150
+Connection ~ 3150 2150
+Wire Wire Line
+	3950 2250 3700 2250
+Connection ~ 3700 2250
 $Comp
 L power:GND #PWR0148
@@
 	5450 3000 5450 2950
 Wire Wire Line
-	5250 3000 4050 3000
-Wire Wire Line
-	4050 3000 4050 2500
-Connection ~ 5250 3000
-Wire Wire Line
-	4050 3000 3500 3000
-Wire Wire Line
-	3500 3000 3500 2400
-Connection ~ 4050 3000
+	3700 3000 3700 2500
+Wire Wire Line
+	3700 3000 3150 3000
+Wire Wire Line
+	3150 3000 3150 2400
+Connection ~ 3700 3000
 $Comp
 L Device:C_Small C701
 U 1 1 60609B81
-P 3200 2850
-F 0 "C701" H 3292 2896 50  0000 L CNN
-F 1 "100n" H 3292 2805 50  0000 L CNN
-F 2 "Capacitor_SMD:C_0603_1608Metric_Pad1.05x0.95mm_HandSolder" H 3200 2850 50  0001 C CNN
-F 3 "https://www.mouser.at/datasheet/2/212/KEM_C1002_X7R_SMD-1102033.pdf" H 3200 2850 50  0001 C CNN
-F 4 "KEMET" H 3200 2850 50  0001 C CNN "Manufacturer"
-F 5 "https://www.mouser.at/ProductDetail/80-C0603C104M4R" H 3200 2850 50  0001 C CNN "Order"
-	1    3200 2850
+P 2850 2850
+F 0 "C701" H 2942 2896 50  0000 L CNN
+F 1 "100n" H 2942 2805 50  0000 L CNN
+F 2 "Capacitor_SMD:C_0603_1608Metric" H 2850 2850 50  0001 C CNN
+F 3 "https://www.mouser.at/datasheet/2/212/KEM_C1002_X7R_SMD-1102033.pdf" H 2850 2850 50  0001 C CNN
+F 4 "KEMET" H 2850 2850 50  0001 C CNN "Manufacturer"
+F 5 "https://www.mouser.at/ProductDetail/80-C0603C104M4R" H 2850 2850 50  0001 C CNN "Order"
+	1    2850 2850
 	1    0    0    -1
 $EndComp
@@
 Wire Wire Line
 	4450 1850 4650 1850
-Text Label 3050 2700 0    50   ~ 0
+Text Label 2700 2700 0    50   ~ 0
 3V3
 Wire Wire Line
-	3050 2700 3200 2700
-Wire Wire Line
-	3200 2700 3200 2750
-Wire Wire Line
-	3200 2950 3200 3000
-Wire Wire Line
-	3200 3000 3500 3000
-Connection ~ 3500 3000
+	2700 2700 2850 2700
+Wire Wire Line
+	2850 2700 2850 2750
+Wire Wire Line
+	2850 2950 2850 3000
+Wire Wire Line
+	2850 3000 3150 3000
+Connection ~ 3150 3000
 Text Label 5600 1450 2    50   ~ 0
 3V3
@@
 F 0 "C705" H 4292 1446 50  0000 L CNN
 F 1 "100n" H 4292 1355 50  0000 L CNN
-F 2 "Capacitor_SMD:C_0603_1608Metric_Pad1.05x0.95mm_HandSolder" H 4200 1400 50  0001 C CNN
+F 2 "Capacitor_SMD:C_0603_1608Metric" H 4200 1400 50  0001 C CNN
 F 3 "https://www.mouser.at/datasheet/2/212/KEM_C1002_X7R_SMD-1102033.pdf" H 4200 1400 50  0001 C CNN
 F 4 "KEMET" H 4200 1400 50  0001 C CNN "Manufacturer"
@@
 F 0 "C703" H 3942 1446 50  0000 L CNN
 F 1 "4.7u" H 3942 1355 50  0000 L CNN
-F 2 "Capacitor_SMD:C_0603_1608Metric_Pad1.05x0.95mm_HandSolder" H 3850 1400 50  0001 C CNN
+F 2 "Capacitor_SMD:C_0805_2012Metric" H 3850 1400 50  0001 C CNN
 F 3 "~" H 3850 1400 50  0001 C CNN
 	1    3850 1400
@@
 F 0 "Q701" V 6792 1350 50  0000 C CNN
 F 1 "DMP2110UW-7" V 6701 1350 50  0000 C CNN
-F 2 "Package_TO_SOT_SMD:SOT-323_SC-70_Handsoldering" H 6650 1450 50  0001 C CNN
+F 2 "Package_TO_SOT_SMD:SOT-323_SC-70" H 6650 1450 50  0001 C CNN
 F 3 "https://www.diodes.com/assets/Datasheets/DMP2110UW.pdf" H 6450 1350 50  0001 C CNN
 F 4 "Diodes Incorporated" H 6450 1350 50  0001 C CNN "Manufacturer"
@@
 F 0 "R704" H 6509 2096 50  0000 L CNN
 F 1 "1k" H 6509 2005 50  0000 L CNN
-F 2 "Resistor_SMD:R_0603_1608Metric_Pad1.05x0.95mm_HandSolder" H 6450 2050 50  0001 C CNN
+F 2 "Resistor_SMD:R_0603_1608Metric" H 6450 2050 50  0001 C CNN
 F 3 "~" H 6450 2050 50  0001 C CNN
 	1    6450 2050
@@
 F 0 "R703" H 6109 1496 50  0000 L CNN
 F 1 "100k" H 6109 1405 50  0000 L CNN
-F 2 "Resistor_SMD:R_0603_1608Metric_Pad1.05x0.95mm_HandSolder" H 6050 1450 50  0001 C CNN
+F 2 "Resistor_SMD:R_0603_1608Metric" H 6050 1450 50  0001 C CNN
 F 3 "https://www.mouser.at/datasheet/2/418/5/NG_DS_9-1773463-9_A-1358566.pdf" H 6050 1450 50  0001 C CNN
 F 4 "TE Connectivity / Holsworthy" H 6050 1450 50  0001 C CNN "Manufacturer"
@@
 F 0 "C706" H 6892 1446 50  0000 L CNN
 F 1 "100n" H 6892 1355 50  0000 L CNN
-F 2 "Capacitor_SMD:C_0603_1608Metric_Pad1.05x0.95mm_HandSolder" H 6800 1400 50  0001 C CNN
+F 2 "Capacitor_SMD:C_0603_1608Metric" H 6800 1400 50  0001 C CNN
 F 3 "https://www.mouser.at/datasheet/2/212/KEM_C1002_X7R_SMD-1102033.pdf" H 6800 1400 50  0001 C CNN
 F 4 "KEMET" H 6800 1400 50  0001 C CNN "Manufacturer"
@@
 F 0 "C707" H 7392 1446 50  0000 L CNN
 F 1 "100n" H 7392 1355 50  0000 L CNN
-F 2 "Capacitor_SMD:C_0603_1608Metric_Pad1.05x0.95mm_HandSolder" H 7300 1400 50  0001 C CNN
+F 2 "Capacitor_SMD:C_0603_1608Metric" H 7300 1400 50  0001 C CNN
 F 3 "https://www.mouser.at/datasheet/2/212/KEM_C1002_X7R_SMD-1102033.pdf" H 7300 1400 50  0001 C CNN
 F 4 "KEMET" H 7300 1400 50  0001 C CNN "Manufacturer"
@@
 Text HLabel 6050 2150 2    50   Input ~ 0
 CTS
+Text Label 4350 2150 0    50   ~ 0
+CHIP_D+
+Text Label 4350 2250 0    50   ~ 0
+CHIP_D-
+Wire Wire Line
+	4150 2150 4650 2150
+Wire Wire Line
+	4150 2250 4650 2250
+Wire Wire Line
+	3700 3000 5250 3000
+Connection ~ 5250 3000
 $EndSCHEMATC

Commit message: added powerflags
Connections:
- no-connect marks 0 -> 3
Changed lines of the file:
@@
 5V
 Wire Wire Line
-	7650 1250 7300 1250
+	7650 1250 7500 1250
 Connection ~ 7300 1250
 Text HLabel 6050 1850 2    50   Output ~ 0
@@
 	3700 3000 5250 3000
 Connection ~ 5250 3000
+NoConn ~ 6050 2350
+NoConn ~ 6050 2450
+NoConn ~ 6050 2550
+$Comp
+L power:PWR_FLAG #FLG0103
+U 1 1 606AA058
+P 7500 1250
+F 0 "#FLG0103" H 7500 1325 50  0001 C CNN
+F 1 "PWR_FLAG" H 7500 1423 50  0000 C CNN
+F 2 "" H 7500 1250 50  0001 C CNN
+F 3 "~" H 7500 1250 50  0001 C CNN
+	1    7500 1250
+	1    0    0    -1
+$EndComp
+Connection ~ 7500 1250
+Wire Wire Line
+	7500 1250 7300 1250
 $EndSCHEMATC

Commit message: minor improvements
Changed lines of the file:
@@
 U 1 1 60606806
 P 4050 2150
-F 0 "R701" V 4100 2300 50  0000 C CNN
+F 0 "R701" V 4100 2350 50  0000 C CNN
 F 1 "27R" V 4100 2000 50  0000 C CNN
 F 2 "Resistor_SMD:R_0603_1608Metric" H 4050 2150 50  0001 C CNN
@@
 U 1 1 6060717E
 P 4050 2250
-F 0 "R702" V 4100 2400 50  0000 C CNN
+F 0 "R702" V 4100 2450 50  0000 C CNN
 F 1 "27R" V 4100 2100 50  0000 C CNN
 F 2 "Resistor_SMD:R_0603_1608Metric" H 4050 2250 50  0001 C CNN
