File: hardware/USB.sch (KiCad schematic (older format))
At the start: 13 parts, among them Q701 DMP2110UW-7, U701 FT230XQ

Commit message: added order references to parts
Parts:
- C702, C704: Manufacturer (none) -> KEMET; Order (none) -> https://www.mouser.at/ProductDetail/KEMET/C0603C470J5RACTU?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
- C703: Manufacturer (none) -> KEMET; Order (none) -> https://www.mouser.at/ProductDetail/KEMET/C0805C475J4RACAUT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
- R701, R702, R704: Manufacturer (none) -> TE Connectivity / Holsworthy; Order (none) -> https://www.mouser.at/ProductDetail/TE-Connectivity-Holswor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
- U701: Manufacturer (none) -> FTDI; Order (none) -> https://www.mouser.at/ProductDetail/FTDI/FT230XQ-R?qs=Gp1Yz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
Changed lines of the file:
@@
 F 2 "Capacitor_SMD:C_0603_1608Metric" H 3150 2300 50  0001 C CNN
 F 3 "~" H 3150 2300 50  0001 C CNN
+F 4 "KEMET" H 3150 2300 50  0001 C CNN "Manufacturer"
+F 5 "https://www.mouser.at/ProductDetail/KEMET/C0603C470J5RACTU?qs=Mv1qlCsH0%252BFrXcCYJrgV0A%3D%3D" H 3150 2300 50  0001 C CNN "Order"
 	1    3150 2300
 	1    0    0    -1
@@
 F 2 "Capacitor_SMD:C_0603_1608Metric" H 3700 2400 50  0001 C CNN
 F 3 "~" H 3700 2400 50  0001 C CNN
+F 4 "KEMET" H 3700 2400 50  0001 C CNN "Manufacturer"
+F 5 "https://www.mouser.at/ProductDetail/KEMET/C0603C470J5RACTU?qs=Mv1qlCsH0%252BFrXcCYJrgV0A%3D%3D" H 3700 2400 50  0001 C CNN "Order"
 	1    3700 2400
 	1    0    0    -1
@@
 F 2 "Package_DFN_QFN:QFN-16-1EP_4x4mm_P0.65mm_EP2.1x2.1mm" H 6700 1650 50  0001 C CNN
 F 3 "https://www.ftdichip.com/Support/Documents/DataSheets/ICs/DS_FT230X.pdf" H 5350 2250 50  0001 C CNN
+F 4 "FTDI" H 5350 2250 50  0001 C CNN "Manufacturer"
+F 5 "https://www.mouser.at/ProductDetail/FTDI/FT230XQ-R?qs=Gp1Yz1mis3VvmXwyDmIHOg%3D%3D" H 5350 2250 50  0001 C CNN "Order"
 	1    5350 2250
 	1    0    0    -1
@@
 F 2 "Resistor_SMD:R_0603_1608Metric" H 4050 2150 50  0001 C CNN
 F 3 "~" H 4050 2150 50  0001 C CNN
+F 4 "TE Connectivity / Holsworthy" H 4050 2150 50  0001 C CNN "Manufacturer"
+F 5 "https://www.mouser.at/ProductDetail/TE-Connectivity-Holsworthy/CRGP0603F27R?qs=wUXugUrL1qwrkVmXivS5zA%3D%3D" H 4050 2150 50  0001 C CNN "Order"
 	1    4050 2150
 	0    -1   -1   0
@@
 F 2 "Resistor_SMD:R_0603_1608Metric" H 4050 2250 50  0001 C CNN
 F 3 "~" H 4050 2250 50  0001 C CNN
+F 4 "TE Connectivity / Holsworthy" H 4050 2250 50  0001 C CNN "Manufacturer"
+F 5 "https://www.mouser.at/ProductDetail/TE-Connectivity-Holsworthy/CRGP0603F27R?qs=wUXugUrL1qwrkVmXivS5zA%3D%3D" H 4050 2250 50  0001 C CNN "Order"
 	1    4050 2250
 	0    -1   -1   0
@@
 F 2 "Capacitor_SMD:C_0805_2012Metric" H 3850 1400 50  0001 C CNN
 F 3 "~" H 3850 1400 50  0001 C CNN
+F 4 "KEMET" H 3850 1400 50  0001 C CNN "Manufacturer"
+F 5 "https://www.mouser.at/ProductDetail/KEMET/C0805C475J4RACAUTO7210?qs=HXFqYaX1Q2wFM9xlsa%252BZZw%3D%3D" H 3850 1400 50  0001 C CNN "Order"
 	1    3850 1400
 	1    0    0    -1
@@
 F 2 "Resistor_SMD:R_0603_1608Metric" H 6450 2050 50  0001 C CNN
 F 3 "~" H 6450 2050 50  0001 C CNN
+F 4 "TE Connectivity / Holsworthy" H 6450 2050 50  0001 C CNN "Manufacturer"
+F 5 "https://www.mouser.at/ProductDetail/TE-Connectivity-Holsworthy/CRGP0603F1K0?qs=sGAEpiMZZMtlubZbdhIBIOInyB5Ysv8sRTd2oyB6aAs%3D" H 6450 2050 50  0001 C CNN "Order"
 	1    6450 2050
 	1    0    0    -1

Commit message: modified bom
Parts:
- C701, C705, C706, C707: MNR (none) -> C0603C104M4RACTU
- C702, C704: MNR (none) -> C0603C470J5RACTU
- C703: MNR (none) -> C0805C475J4RACAUTO7210
- Q701: MNR (none) -> DMP2110UW-7
- R701, R702: MNR (none) -> CRGP0603F27R
- R703: MNR (none) -> CRGP0603F100K
- R704: MNR (none) -> CRGP0603F1K0
- U701: MNR (none) -> FT230XQ-R
Changed lines of the file:
@@
 F 4 "KEMET" H 3150 2300 50  0001 C CNN "Manufacturer"
 F 5 "https://www.mouser.at/ProductDetail/KEMET/C0603C470J5RACTU?qs=Mv1qlCsH0%252BFrXcCYJrgV0A%3D%3D" H 3150 2300 50  0001 C CNN "Order"
+F 6 "C0603C470J5RACTU" H 3150 2300 50  0001 C CNN "MNR"
 	1    3150 2300
 	1    0    0    -1
@@
 F 4 "KEMET" H 3700 2400 50  0001 C CNN "Manufacturer"
 F 5 "https://www.mouser.at/ProductDetail/KEMET/C0603C470J5RACTU?qs=Mv1qlCsH0%252BFrXcCYJrgV0A%3D%3D" H 3700 2400 50  0001 C CNN "Order"
+F 6 "C0603C470J5RACTU" H 3700 2400 50  0001 C CNN "MNR"
 	1    3700 2400
 	1    0    0    -1
@@
 F 4 "FTDI" H 5350 2250 50  0001 C CNN "Manufacturer"
 F 5 "https://www.mouser.at/ProductDetail/FTDI/FT230XQ-R?qs=Gp1Yz1mis3VvmXwyDmIHOg%3D%3D" H 5350 2250 50  0001 C CNN "Order"
+F 6 "FT230XQ-R" H 5350 2250 50  0001 C CNN "MNR"
 	1    5350 2250
 	1    0    0    -1
@@
 F 4 "TE Connectivity / Holsworthy" H 4050 2150 50  0001 C CNN "Manufacturer"
 F 5 "https://www.mouser.at/ProductDetail/TE-Connectivity-Holsworthy/CRGP0603F27R?qs=wUXugUrL1qwrkVmXivS5zA%3D%3D" H 4050 2150 50  0001 C CNN "Order"
+F 6 "CRGP0603F27R" H 4050 2150 50  0001 C CNN "MNR"
 	1    4050 2150
 	0    -1   -1   0
@@
 F 4 "TE Connectivity / Holsworthy" H 4050 2250 50  0001 C CNN "Manufacturer"
 F 5 "https://www.mouser.at/ProductDetail/TE-Connectivity-Holsworthy/CRGP0603F27R?qs=wUXugUrL1qwrkVmXivS5zA%3D%3D" H 4050 2250 50  0001 C CNN "Order"
+F 6 "CRGP0603F27R" H 4050 2250 50  0001 C CNN "MNR"
 	1    4050 2250
 	0    -1   -1   0
@@
 F 4 "KEMET" H 2850 2850 50  0001 C CNN "Manufacturer"
 F 5 "https://www.mouser.at/ProductDetail/80-C0603C104M4R" H 2850 2850 50  0001 C CNN "Order"
+F 6 "C0603C104M4RACTU" H 2850 2850 50  0001 C CNN "MNR"
 	1    2850 2850
 	1    0    0    -1
@@
 F 4 "KEMET" H 4200 1400 50  0001 C CNN "Manufacturer"
 F 5 "https://www.mouser.at/ProductDetail/80-C0603C104M4R" H 4200 1400 50  0001 C CNN "Order"
+F 6 "C0603C104M4RACTU" H 4200 1400 50  0001 C CNN "MNR"
 	1    4200 1400
 	1    0    0    -1
@@
 F 4 "KEMET" H 3850 1400 50  0001 C CNN "Manufacturer"
 F 5 "https://www.mouser.at/ProductDetail/KEMET/C0805C475J4RACAUTO7210?qs=HXFqYaX1Q2wFM9xlsa%252BZZw%3D%3D" H 3850 1400 50  0001 C CNN "Order"
+F 6 "C0805C475J4RACAUTO7210" H 3850 1400 50  0001 C CNN "MNR"
 	1    3850 1400
 	1    0    0    -1
@@
 F 4 "Diodes Incorporated" H 6450 1350 50  0001 C CNN "Manufacturer"
 F 5 "https://www.mouser.at/ProductDetail/Diodes-Incorporated/DMP2110UW-7?qs=bZr6mbWTK5lZsAURvLPe3w%3D%3D" H 6450 1350 50  0001 C CNN "Order"
+F 6 "DMP2110UW-7" H 6450 1350 50  0001 C CNN "MNR"
 	1    6450 1350
 	0    1    -1   0
@@
 F 4 "TE Connectivity / Holsworthy" H 6450 2050 50  0001 C CNN "Manufacturer"
 F 5 "https://www.mouser.at/ProductDetail/TE-Connectivity-Holsworthy/CRGP0603F1K0?qs=sGAEpiMZZMtlubZbdhIBIOInyB5Ysv8sRTd2oyB6aAs%3D" H 6450 2050 50  0001 C CNN "Order"
+F 6 "CRGP0603F1K0" H 6450 2050 50  0001 C CNN "MNR"
 	1    6450 2050
 	1    0    0    -1
@@
 F 4 "TE Connectivity / Holsworthy" H 6050 1450 50  0001 C CNN "Manufacturer"
 F 5 "https://www.mouser.at/ProductDetail/279-CRGP0603F100K" H 6050 1450 50  0001 C CNN "Order"
+F 6 "CRGP0603F100K" H 6050 1450 50  0001 C CNN "MNR"
 	1    6050 1450
 	1    0    0    -1
@@
 F 4 "KEMET" H 6800 1400 50  0001 C CNN "Manufacturer"
 F 5 "https://www.mouser.at/ProductDetail/80-C0603C104M4R" H 6800 1400 50  0001 C CNN "Order"
+F 6 "C0603C104M4RACTU" H 6800 1400 50  0001 C CNN "MNR"
 	1    6800 1400
 	1    0    0    -1
@@
 F 4 "KEMET" H 7300 1400 50  0001 C CNN "Manufacturer"
 F 5 "https://www.mouser.at/ProductDetail/80-C0603C104M4R" H 7300 1400 50  0001 C CNN "Order"
+F 6 "C0603C104M4RACTU" H 7300 1400 50  0001 C CNN "MNR"
 	1    7300 1400
 	1    0    0    -1

Commit message: Fixed two hardware issues.
Issue 1: Swapped USB D+/- lines
Issue 2: Wrong schematic smybol for power switch
Connections:
- net CHIP_D+: now also R702.2, U701.6 (USBDP); no longer R701.2, U701.7 (USBDM)
- net CHIP_D-: now also R701.2, U701.7 (USBDM); no longer R702.2, U701.6 (USBDP)
- net D+: now also C704.1, R702.1; no longer C702.1, R701.1
- net D-: now also C702.1, R701.1; no longer C704.1, R702.1
Changed lines of the file:
@@
 Text HLabel 3700 1250 0    50   Input ~ 0
 VBUS
+Text HLabel 3650 2250 0    50   Input ~ 0
+D+
 Text HLabel 3100 2150 0    50   Input ~ 0
-D+
-Text HLabel 3650 2250 0    50   Input ~ 0
 D-
 $Comp
@@
 Text HLabel 6050 2150 2    50   Input ~ 0
 CTS
+Text Label 4350 2250 0    50   ~ 0
+CHIP_D+
 Text Label 4350 2150 0    50   ~ 0
-CHIP_D+
-Text Label 4350 2250 0    50   ~ 0
 CHIP_D-
 Wire Wire Line
